File: flight_controller_pcb/_autosave-flight_controller_pcb.kicad_pcb (KiCad board)
At the start: 4 copper layers, 27 x 32 mm, 69 parts, among them J1 Conn_01x08, J2 Conn_01x05, J3 Conn_01x02, U1 NRF24L01P-R7, U10 SN74LVC2T45YZP, U11 SN74LVC1T45DRL, U2 TPS62162, U3 STM32F411CEUx, U4 RFX2401C, U5 BMP390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

Commit message: pcb routing
Parts:
- moved C2 99.9 mm to (110.2, 149.8)
- moved C3 97.6 mm to (110.2, 148.5)
- moved C4 96.7 mm to (114.2, 144.3), turned to 180 degrees
- moved R1 89.5 mm to (114.2, 146.3)
- moved U1 18.7 mm to (109.4, 144.8)
Routing:
- net +3.3V: track 23.0 -> 38.9 mm
- net /SPI1_MOSI: track 3.84 -> 0.00 mm, vias 1 -> 0
- net /SPI1_SCK: track 3.32 -> 0.36 mm, vias 2 -> 0
- net Net-(U1-IREF): track 0.00 -> 2.81 mm, vias 0 -> 2
- net Net-(U1-DVDD): track 0.00 -> 2.60 mm
- net GND: track 0.00 -> 1.12 mm, vias 0 -> 1
